Commit message: fix: make OrbiBot visible in Gazebo (dark chassis color)
Chassis was rgba(0.8,0.8,0.8) — same as gray ground plane — causing the
robot to be invisible in Gazebo GUI despite being physically present.
Changed to dark (0.1,0.1,0.1) + added Gazebo/DarkGrey material tag
(gz-sim ignores URDF material colors without explicit <gazebo> override).

File: src/orbibot_description/urdf/orbibot.urdf.xacro (robot description, xacro)
@@ -43,5 +43,5 @@
       </geometry>
       <material name="chassis_material">
-        <color rgba="0.8 0.8 0.8 1.0"/>
+        <color rgba="0.1 0.1 0.1 1.0"/>
       </material>
     </visual>
@@ -301,4 +301,8 @@
     </sensor>
   </gazebo>
+  <!-- Chassis color for Gazebo (URDF material colors are ignored by gz-sim) -->
+  <gazebo reference="base_link">
+    <material>Gazebo/DarkGrey</material>
+  </gazebo>
   <!-- Wheel friction properties (improves sim driving feel) -->
   <gazebo reference="wheel_front_left_link">

Commit message: change rviz robot color

File: src/orbibot_description/urdf/orbibot.urdf.xacro (robot description, xacro)
@@ -43,5 +43,5 @@
       </geometry>
       <material name="chassis_material">
-        <color rgba="0.1 0.1 0.1 1.0"/>
+        <color rgba="0.85 0.45 0.05 1.0"/>
       </material>
     </visual>
@@ -303,5 +303,5 @@
   <!-- Chassis color for Gazebo (URDF material colors are ignored by gz-sim) -->
   <gazebo reference="base_link">
-    <material>Gazebo/DarkGrey</material>
+    <material>Gazebo/Orange</material>
   </gazebo>
   <!-- Wheel friction properties (improves sim driving feel) -->
