Commit message: fix(description): the IMU is mounted 90 degrees out — imu_joint said rpy="0 0 0"
The ICM-20948's axes are not aligned with the chassis: the sensor's +X points
along the robot's LEFT (base_link +Y). The board is not rotated -- the chip on
it is -- which is why nothing looked wrong to the eye, and why the URDF has
claimed rpy="0 0 0" for as long as it has existed. Roll and pitch were swapped
everywhere downstream of the IMU.

Proven three independent ways before the change, verified after. test-report.md
section 9.9 has every number.

1. Physical pitch shows up as sensor ROLL. Named tilts kept contradicting each
   other because "lift the left side" depends on where the operator stands; the
   test that worked used a visible feature instead of a direction -- the camera.
   Camera end up: roll +21.86, +23.45, +23.33. Camera end down: -22.24, -21.01.
   Pitch moved by ~1 degree throughout. Three separate holds, both directions.

2. The frame is a ROTATION, not a reflection. A roll/pitch swap could equally
   have been X and Y exchanged without a sign change -- left-handed, impossible
   from mounting, and therefore an index bug in firmware or driver rather than a
   URDF error. The two differ in handedness, and handedness shows up in a yaw
   rotation, which can be specified without the words left or right:

     clockwise from above    gyro Z  -25.38 and -41.25 deg/s   yaw -22.00, -90.13
     counter-clockwise       gyro Z  +44.86 deg/s              yaw +84.04

   Sign follows direction, so right-handed, so a rotation, so the URDF. In a
   right-handed frame nose-up -> roll positive happens for exactly one
   orientation: +90 degrees.

3. End-to-end after the fix. TF reports base_link <- imu_link yaw +90.00. With
   the camera end held up the topic still says roll +8.32 ("left side up"),
   while the same data resolved into base_link says pitch +8.32 -- NOSE UP.

Impact before the fix was small and about to stop being small: imu0_config
fuses yaw and vyaw only, imu0_relative cancels a constant yaw offset, and
angular velocity about Z is invariant under a Z-rotation, so the EKF's
arithmetic was unaffected. It would have started mattering the moment
two_d_mode was disabled, accel fusion enabled, roll/pitch used for a tilt check,
or anyone read /imu/data_filtered directly. RViz was wrong throughout.

This also corrects a wrong conclusion I committed earlier today. LOC-1 said
"the axes are fine", closed on the sensor reading roll -0.935 and the operator
saying the right side looked high -- two observations agreeing. They agreed by
coincidence: the operator's FIRST description was "the rear is raised", a pitch,
and the second was hedged. Translated through the rotation, roll -0.935 means
rear raised 0.94 degrees with no side tilt, which is what was said first. The
correction is written into LOC-1 rather than quietly replacing the text.

Section 9.7's drift analysis is unaffected -- it was computed entirely in the
sensor frame and is self-consistent there. Only the labels move: the leaking
term is the sensor Y gyro bias, the robot's roll axis, leaking through a rear-up
pitch. The 0.47 % model agreement and the 5.6x available from levelling stand.

Adds imu_base_frame.py, which resolves /imu/data_filtered into base_link using
TF and prints both, so this class of error is visible rather than inferred.

Also fixes seven stale figures in the localization README left by this morning's
EKF 25 -> 50 Hz change, and the /odom rate, which is on-change plus a 0.5 s
heartbeat rather than 20 Hz.

File: src/orbibot_description/urdf/orbibot.urdf.xacro (robot description, xacro)
@@ -180,9 +180,16 @@
   </joint>
   <link name="camera_depth_optical_frame"/>
-  <!-- IMU sensor -->
+  <!-- IMU sensor.
+       The ICM-20948's axes are NOT aligned with the chassis: the sensor's +X
+       points along the robot's LEFT (base_link +Y), i.e. the frame is rotated
+       +90 deg about Z. Measured 2026-08-04, three independent ways —
+       test-report.md 9.9. Until then this joint claimed rpy="0 0 0" and roll
+       and pitch were silently swapped everywhere downstream.
+       Do not "simplify" this back to zero because the board looks square-on in
+       the chassis. The board is not rotated; the chip on it is. -->
   <joint name="imu_joint" type="fixed">
     <parent link="base_link"/>
     <child link="imu_link"/>
-    <origin xyz="0.0 0.0 0.02" rpy="0 0 0"/>
+    <origin xyz="0.0 0.0 0.02" rpy="0 0 1.5707963"/>
   </joint>
   <link name="imu_link">
